File: rp2040zero_modxo.kicad_pcb (KiCad board)
At the start: 2 copper layers, 36.5 x 30.5 mm, 6 parts, among them J1 Conn_02x08_Odd_Even

Commit message: Added gitmodule rp2040zero footprint
Parts:
- U1: footprint RP2040:RP2040 Zero -> rp2040zero_fp:RP2040 Zero
Connections:
- U1 pad 1: (no net) -> unconnected-(U1A-GPIO0-Pad1)
- U1 pad 10: (no net) -> unconnected-(U1A-GPIO9-Pad10)
- U1 pad 11: (no net) -> unconnected-(U1A-GPIO10-Pad11)
- U1 pad 12: (no net) -> unconnected-(U1A-GPIO11-Pad12)
- U1 pad 13: (no net) -> unconnected-(U1A-GPIO12-Pad13)
- U1 pad 14: (no net) -> unconnected-(U1A-GPIO13-Pad14)
- U1 pad 15: (no net) -> unconnected-(U1A-GPIO14-Pad15)
- U1 pad 16: (no net) -> unconnected-(U1A-GPIO15-Pad16)
- U1 pad 17: (no net) -> unconnected-(U1A-GPIO26-Pad17)
- U1 pad 18: (no net) -> unconnected-(U1A-GPIO27-Pad18)
- U1 pad 19: (no net) -> unconnected-(U1A-GPIO28-Pad19)
- U1 pad 2: (no net) -> unconnected-(U1A-GPIO1-Pad2)
- U1 pad 20: (no net) -> unconnected-(U1A-GPIO29-Pad20)
- U1 pad 21: (no net) -> unconnected-(U1A-3V3-Pad21)
- U1 pad 3: (no net) -> unconnected-(U1A-GPIO2-Pad3)
- U1 pad 4: (no net) -> unconnected-(U1A-GPIO3-Pad4)
- U1 pad 5: (no net) -> unconnected-(U1A-GPIO4-Pad5)
- U1 pad 6: (no net) -> unconnected-(U1A-GPIO5-Pad6)
- U1 pad 7: (no net) -> unconnected-(U1A-GPIO6-Pad7)
- U1 pad 8: (no net) -> unconnected-(U1A-GPIO7-Pad8)
- U1 pad 9: (no net) -> unconnected-(U1A-GPIO8-Pad9)
Changed lines of the file:
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@@
 	(net 13 "/LAD3")
 	(net 14 "/D0")
-	(footprint "RP2040:RP2040 Zero"
+	(net 15 "unconnected-(U1A-GPIO27-Pad18)")
+	(net 16 "unconnected-(U1A-GPIO26-Pad17)")
+	(net 17 "unconnected-(U1A-GPIO28-Pad19)")
+	(net 18 "unconnected-(U1A-GPIO7-Pad8)")
+	(net 19 "unconnected-(U1A-3V3-Pad21)")
+	(net 20 "unconnected-(U1A-GPIO14-Pad15)")
+	(net 21 "unconnected-(U1A-GPIO6-Pad7)")
+	(net 22 "unconnected-(U1A-GPIO0-Pad1)")
+	(net 23 "unconnected-(U1A-GPIO1-Pad2)")
+	(net 24 "unconnected-(U1A-GPIO29-Pad20)")
+	(net 25 "unconnected-(U1A-GPIO2-Pad3)")
+	(net 26 "unconnected-(U1A-GPIO3-Pad4)")
+	(net 27 "unconnected-(U1A-GPIO9-Pad10)")
+	(net 28 "unconnected-(U1A-GPIO4-Pad5)")
+	(net 29 "unconnected-(U1A-GPIO10-Pad11)")
+	(net 30 "unconnected-(U1A-GPIO12-Pad13)")
+	(net 31 "unconnected-(U1A-GPIO13-Pad14)")
+	(net 32 "unconnected-(U1A-GPIO8-Pad9)")
+	(net 33 "unconnected-(U1A-GPIO11-Pad12)")
+	(net 34 "unconnected-(U1A-GPIO5-Pad6)")
+	(net 35 "unconnected-(U1A-GPIO15-Pad16)")
+	(footprint "rp2040zero_fp:RP2040 Zero"
 		(layer "F.Cu")
 		(at 138.38 71.59)
@@
 			)
 		)
-		(property "Footprint" "RP2040:RP2040 Zero"
+		(property "Footprint" "rp2040zero_fp:RP2040 Zero"
 			(at 0 -23.5 0)
 			(unlocked yes)
@@
 			(size 3.1405 1.521)
 			(layers "F.Cu" "F.Paste" "F.Mask")
+			(net 22 "unconnected-(U1A-GPIO0-Pad1)")
+			(pinfunction "GPIO0")
+			(pintype "bidirectional+no_connect")
 		)
 		(pad "2" smd rect
@@
 			(size 3.1405 1.521)
 			(layers "F.Cu" "F.Paste" "F.Mask")
+			(net 23 "unconnected-(U1A-GPIO1-Pad2)")
+			(pinfunction "GPIO1")
+			(pintype "bidirectional+no_connect")
 		)
 		(pad "3" smd rect
@@
 			(size 3.1405 1.521)
 			(layers "F.Cu" "F.Paste" "F.Mask")
+			(net 25 "unconnected-(U1A-GPIO2-Pad3)")
+			(pinfunction "GPIO2")
+			(pintype "bidirectional+no_connect")
 		)
 		(pad "4" smd rect
@@
 			(size 3.1405 1.5505)
 			(layers "F.Cu" "F.Paste" "F.Mask")
+			(net 26 "unconnected-(U1A-GPIO3-Pad4)")
+			(pinfunction "GPIO3")
+			(pintype "bidirectional+no_connect")
 		)
 		(pad "5" smd rect
@@
 			(size 3.1405 1.5105)
 			(layers "F.Cu" "F.Paste" "F.Mask")
+			(net 28 "unconnected-(U1A-GPIO4-Pad5)")
+			(pinfunction "GPIO4")
+			(pintype "bidirectional+no_connect")
 		)
 		(pad "6" smd rect
@@
 			(size 3.1405 1.521)
 			(layers "F.Cu" "F.Paste" "F.Mask")
+			(net 34 "unconnected-(U1A-GPIO5-Pad6)")
+			(pinfunction "GPIO5")
+			(pintype "bidirectional+no_connect")
 		)
 		(pad "7" smd rect
@@
 			(size 3.1405 1.521)
 			(layers "F.Cu" "F.Paste" "F.Mask")
+			(net 21 "unconnected-(U1A-GPIO6-Pad7)")
+			(pinfunction "GPIO6")
+			(pintype "bidirectional+no_connect")
 		)
 		(pad "8" smd rect
@@
 			(size 3.1405 1.521)
 			(layers "F.Cu" "F.Paste" "F.Mask")
+			(net 18 "unconnected-(U1A-GPIO7-Pad8)")
+			(pinfunction "GPIO7")
+			(pintype "bidirectional+no_connect")
 		)
 		(pad "9" thru_hole circle
@@
 			(layers "*.Cu" "*.Mask")
 			(remove_unused_layers no)
+			(net 32 "unconnected-(U1A-GPIO8-Pad9)")
+			(pinfunction "GPIO8")
+			(pintype "bidirectional+no_connect")
 			(thermal_bridge_angle 90)
 		)
@@
 			(size 1.521 3.3705)
 			(layers "F.Cu" "F.Paste" "F.Mask")
+			(net 27 "unconnected-(U1A-GPIO9-Pad10)")
+			(pinfunction "GPIO9")
+			(pintype "bidirectional+no_connect")
 		)
 		(pad "11" smd rect
@@
 			(size 1.521 3.3705)
 			(layers "F.Cu" "F.Paste" "F.Mask")
+			(net 29 "unconnected-(U1A-GPIO10-Pad11)")
+			(pinfunction "GPIO10")
+			(pintype "bidirectional+no_connect")
 		)
 		(pad "12" smd rect
@@
 			(size 1.521 3.3705)
 			(layers "F.Cu" "F.Paste" "F.Mask")
+			(net 33 "unconnected-(U1A-GPIO11-Pad12)")
+			(pinfunction "GPIO11")
+			(pintype "bidirectional+no_connect")
 		)
 		(pad "13" smd rect
@@
 			(size 1.521 3.3705)
 			(layers "F.Cu" "F.Paste" "F.Mask")
+			(net 30 "unconnected-(U1A-GPIO12-Pad13)")
+			(pinfunction "GPIO12")
+			(pintype "bidirectional+no_connect")
 		)
 		(pad "14" smd rect
@@
 			(size 1.521 3.3705)
 			(layers "F.Cu" "F.Paste" "F.Mask")
+			(net 31 "unconnected-(U1A-GPIO13-Pad14)")
+			(pinfunction "GPIO13")
+			(pintype "bidirectional+no_connect")
 		)
 		(pad "15" smd rect
@@
 			(size 3.1405 1.521)
 			(layers "F.Cu" "F.Paste" "F.Mask")
+			(net 20 "unconnected-(U1A-GPIO14-Pad15)")
+			(pinfunction "GPIO14")
+			(pintype "bidirectional+no_connect")
 		)
 		(pad "16" smd rect
@@
 			(size 3.1405 1.521)
 			(layers "F.Cu" "F.Paste" "F.Mask")
+			(net 35 "unconnected-(U1A-GPIO15-Pad16)")
+			(pinfunction "GPIO15")
+			(pintype "bidirectional+no_connect")
 		)
 		(pad "17" smd rect
@@
 			(size 3.1405 1.521)
 			(layers "F.Cu" "F.Paste" "F.Mask")
+			(net 16 "unconnected-(U1A-GPIO26-Pad17)")
+			(pinfunction "GPIO26")
+			(pintype "bidirectional+no_connect")
 		)
 		(pad "18" smd rect
@@
 			(size 3.1405 1.521)
 			(layers "F.Cu" "F.Paste" "F.Mask")
+			(net 15 "unconnected-(U1A-GPIO27-Pad18)")
+			(pinfunction "GPIO27")
+			(pintype "bidirectional+no_connect")
 		)
 		(pad "19" smd rect
@@
 			(size 3.1405 1.5105)
 			(layers "F.Cu" "F.Paste" "F.Mask")
+			(net 17 "unconnected-(U1A-GPIO28-Pad19)")
+			(pinfunction "GPIO28")
+			(pintype "bidirectional+no_connect")
 		)
 		(pad "20" smd rect
@@
 			(size 3.1405 1.5505)
 			(layers "F.Cu" "F.Paste" "F.Mask")
+			(net 24 "unconnected-(U1A-GPIO29-Pad20)")
+			(pinfunction "GPIO29")
+			(pintype "bidirectional+no_connect")
 		)
 		(pad "21" thru_hole circle
@@
 			(layers "*.Cu" "*.Mask")
 			(remove_unused_layers no)
+			(net 19 "unconnected-(U1A-3V3-Pad21)")
+			(pinfunction "3V3")
+			(pintype "power_out+no_connect")
 		)
 		(pad "22" thru_hole circle
