File: rp2040zero_modxo.kicad_sch (KiCad schematic)
At the start: 6 parts, among them J1 Conn_02x08_Odd_Even

Commit message: Added gitmodule rp2040zero footprint
Parts:
- U1: footprint RP2040:RP2040 Zero -> rp2040zero_fp:RP2040 Zero
- U1: footprint RP2040:RP2040 Zero -> rp2040zero_fp:RP2040 Zero; symbol RP2040 Zero:RP2040_Zero -> rp2040zero_fp:RP2040_Zero
Changed lines of the file:
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@@
 			)
 		)
-		(property "Footprint" "RP2040:RP2040 Zero"
+		(property "Footprint" "rp2040zero_fp:RP2040 Zero"
 			(at 30.48 21.59 0)
 			(effects
@@
 		(instances
 			(project ""
+				(path "/5c6b4335-7a83-41c6-94b0-4b7942a7378d"
+					(reference "U1")
+					(unit 1)
+				)
+			)
+			(project ""
 				(path "/de6b75b6-5171-4868-8151-c2bba6d8be62"
 					(reference "U1")
@@
 	)
 	(symbol
-		(lib_id "RP2040 Zero:RP2040_Zero")
+		(lib_id "rp2040zero_fp:RP2040_Zero")
 		(at 30.48 81.28 0)
 		(unit 2)
@@
 			)
 		)
-		(property "Footprint" "RP2040:RP2040 Zero"
+		(property "Footprint" "rp2040zero_fp:RP2040 Zero"
 			(at 30.48 81.28 0)
 			(effects
